File: navigator.kicad_pcb (KiCad board)
At the start: 2 copper layers, 42.1 x 38.7 mm, 29 parts, among them J101 SWD, J102 3V3, J103 5V, J104 GND, J105 INPUT, J106 5V, J107 GND, U101 STM32G030F6Px, U102 5501

Commit message: wip
Parts:
- removed D102: LED_Small, LED_SMD:LED_1206_3216Metric
- removed U101: STM32G030F6Px, Package_SO:TSSOP-20_4.4x6.5mm_P0.65mm
- added D104: D_Schottky_Small, Diode_SMD:D_SOD-323, F.Cu at (86.0, 57.9)
- added JP102: Pu/Pd, Jumper:SolderJumper-3_P1.3mm_Open_RoundedPad1.0x1.5mm, F.Cu at (83.1, 58.3)
- added JP103: debug, Jumper:SolderJumper-2_P1.3mm_Open_Pad1.0x1.5mm, F.Cu at (80.7, 65.8)
- added U103: STM32G030J6Mx, Package_SO:SOIC-8_3.9x4.9mm_P1.27mm, F.Cu at (85.8, 67.2)
- D101: value BZX84Cxx -> LED_Small; footprint Package_TO_SOT_SMD:SOT-23 -> LED_SMD:LED_1206_3216Metric
- R104: value 1K -> 10K
- R105: value 1K -> 100
- moved J104 14.9 mm to (82.7, 82.6)
- moved J102 14.6 mm to (90.7, 71.8), turned to 90 degrees
- moved C101 11.7 mm to (90.5, 67.3), turned to 90 degrees
- moved R103 10.8 mm to (80.6, 62.3), turned to 90 degrees
- moved J101 9.80 mm to (83.5, 71.8), turned to 90 degrees
- moved R102 8.81 mm to (90.6, 58.2), turned to 0 degrees
- moved R106 8.28 mm to (83.1, 62.3)
- moved R105 8.03 mm to (86.0, 61.4), turned to -90 degrees
- moved R104 7.58 mm to (83.1, 54.1)
- moved J107 5.41 mm to (95.8, 82.7)
- moved R101 5.26 mm to (90.6, 60.2), turned to 0 degrees
- moved D101 2.80 mm to (76.2, 59.4)
- moved J105 2.58 mm to (86.1, 54.3)
Connections:
- D101 pad 2: unconnected-(D101-NC-Pad2) -> Net-(D101-A)
- J105 pad 1: Net-(J105-Pin_1) -> Net-(D104-K)
- R101 pad 1: /USART1_TX -> /USART2_TX
- R103 pad 1: /3V3 -> Net-(JP103-A)
- R103 pad 2: Net-(U101-NRST) -> Net-(D101-A)
- R104 pad 1: Net-(J105-Pin_1) -> GND
- R104 pad 2: /INPUT -> Net-(JP102-A)
- R105 pad 1: Net-(J105-Pin_1) -> Net-(D104-A)
- R105 pad 2: Net-(D102-A) -> /INPUT
- R106 pad 1: Net-(J105-Pin_1) -> Net-(JP102-B)
Routing:
- net Net-(J105-Pin_1): track 14.7 -> 0.00 mm
- net Net-(BT101-TXD): track 13.4 -> 2.34 mm
- net /USART1_RX: track 3.33 -> 14.3 mm
- net /3V3: track 57.5 -> 66.2 mm
- net /INPUT: track 13.9 -> 6.58 mm
- net Net-(BT101-RXD): track 9.30 -> 2.65 mm
- net Net-(D104-K): track 0.00 -> 6.01 mm
- net /5V: track 36.4 -> 30.5 mm, vias 2 -> 1
- net Net-(U101-NRST): track 5.77 -> 0.00 mm
- net /USART2_TX: track 0.00 -> 5.74 mm
- net Net-(D101-A): track 0.00 -> 4.67 mm
- net Net-(JP103-A): track 0.00 -> 4.44 mm
- net /USART1_TX: track 3.04 -> 0.00 mm
- net /SWDIO: track 3.46 -> 5.92 mm
- net Net-(JP102-A): track 0.00 -> 1.85 mm
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- added copper zone on B.Cu, net GND

Commit message: Production ready
Parts:
- removed JP102: Pu/Pd, Jumper:SolderJumper-3_P1.3mm_Open_RoundedPad1.0x1.5mm
- added C106: 1uF, Capacitor_SMD:C_0805_2012Metric, F.Cu at (94.5, 64.2)
- added C107: 10uF, Capacitor_SMD:C_0805_2012Metric, F.Cu at (83.8, 74.8)
- added C108: 10uF, Capacitor_SMD:C_0805_2012Metric, F.Cu at (85.9, 74.8)
- added C109: 0.01uF, Capacitor_SMD:C_0603_1608Metric, F.Cu at (90.7, 81.8)
- added D102: SS14FL, Diode_SMD:D_SMF, F.Cu at (85.1, 79.4)
- added L101: 22uH, inductor:FNR5040S220MT, F.Cu at (77.6, 79.0)
- added LOGO101: ~, logo:logo_15x9, B.Cu at (103.5, 58.7)
- added Q101: IRLML9303TRPBF, Package_TO_SOT_SMD:SOT-23, F.Cu at (94.2, 84.3)
- added R109: 10K, Resistor_SMD:R_0603_1608Metric, F.Cu at (93.7, 81.8)
- added R111: 500, Resistor_SMD:R_0805_2012Metric, F.Cu at (78.0, 70.6)
- added R112: 10K, Resistor_SMD:R_0805_2012Metric, F.Cu at (81.4, 70.5)
- added R113: 200, Resistor_SMD:R_0805_2012Metric, F.Cu at (80.8, 56.2)
- added U101: LTV-817S, Package_DIP:SMDIP-4_W9.53mm, F.Cu at (80.0, 63.4)
- C105: value 4.7uF -> 0.1uF
- D104: value D_Schottky_Small -> BZT52C16S
- J103: value 5V -> Vinn
- J106: value 5V -> SensorV
- R104: value 10K -> 100K; footprint Resistor_SMD:R_0805_2012Metric -> Resistor_SMD:R_0603_1608Metric
- R105: value 100 -> 28K; footprint Resistor_SMD:R_0805_2012Metric -> Resistor_SMD:R_0603_1608Metric
- R106: value 10K -> 8K45; footprint Resistor_SMD:R_0805_2012Metric -> Resistor_SMD:R_0603_1608Metric
- U102: value 5501 -> LMR16006Y; footprint Package_TO_SOT_SMD:TO-252-3_TabPin2 -> Package_TO_SOT_SMD:SOT-23-6
- moved R104 29.5 mm to (82.6, 83.6), turned to 180 degrees
- moved D104 26.9 mm to (91.2, 84.3), turned to 90 degrees
- moved J107 26.3 mm to (75.0, 66.7)
- moved R105 24.2 mm to (76.1, 83.4)
- moved R106 21.8 mm to (77.6, 83.4), turned to 90 degrees
- moved J104 21.7 mm to (104.3, 84.3)
- moved J106 17.3 mm to (75.0, 70.3)
- moved J105 14.1 mm to (75.0, 63.1)
- moved D101 12.4 mm to (84.9, 50.6), turned to -90 degrees
- moved C105 11.3 mm to (76.5, 79.3), turned to 90 degrees
- moved JP103 10.4 mm to (87.6, 58.0), turned to 0 degrees
- moved R103 7.85 mm to (84.9, 55.7)
- moved J103 7.37 mm to (98.1, 84.3)
- moved J101 5.17 mm to (87.5, 68.6)
- moved C104 3.78 mm to (84.4, 81.6), turned to 0 degrees
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Connections:
- C104 pad 1: /5V -> /Vin
- C105 pad 1: /3V3 -> Net-(U102-CB)
- C105 pad 2: GND -> Net-(D102-K)
- D104 pad 1: Net-(D104-K) -> /Vin
- J103 pad 1: /5V -> Net-(J103-Pin_1)
- J105 pad 1: Net-(D104-K) -> Net-(J105-Pin_1)
- J106 pad 1: /5V -> /Vin
- R104 pad 1: GND -> /Vin
- R104 pad 2: Net-(JP102-A) -> Net-(U102-~{SHDN})
- R105 pad 1: Net-(D104-A) -> /3V3
- R105 pad 2: /INPUT -> Net-(U102-FB)
- R106 pad 1: Net-(JP102-B) -> Net-(U102-FB)
- R106 pad 2: /5V -> GND
- U102 pad 1: /5V -> Net-(U102-CB)
- U102 pad 3: /3V3 -> Net-(U102-FB)
- U103 pad 5: Net-(JP103-A) -> /SIGNAL
- U103 pad 6: /INPUT -> Net-(JP103-A)
Routing:
- net /Vin: track 0.00 -> 45.2 mm, vias 0 -> 4
- net /5V: track 30.5 -> 0.00 mm, vias 1 -> 0
- net /3V3: track 66.2 -> 79.7 mm, vias 0 -> 2
- net Net-(J105-Pin_1): track 0.00 -> 12.6 mm
- net /SIGNAL: track 0.00 -> 8.92 mm
- net /INPUT: track 6.58 -> 0.00 mm
- net Net-(D104-K): track 6.01 -> 0.00 mm
- net Net-(JP103-A): track 4.44 -> 10.3 mm
- net Net-(U102-FB): track 0.00 -> 4.45 mm
- net Net-(R111-Pad2): track 0.00 -> 3.72 mm
- net Net-(D104-A): track 1.53 -> 4.99 mm
- net Net-(J103-Pin_1): track 0.00 -> 2.98 mm
- net Net-(BT101-LED1): track 3.80 -> 6.74 mm
- net Net-(R113-Pad2): track 0.00 -> 2.87 mm
- net Net-(U102-CB): track 0.00 -> 2.78 mm
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- added copper zone on F.Cu, net /3V3
- added copper zone on F.Cu, net Net-(D102-K)
Other:
- board text added: "3V3"
- board text added: "GND"
- board text added: "SWD"
- board text added: "SWDCLK"
- board text added: "SWDIO"
- board text added: "ВХОД 5-60В - +"
- board text added: "ВЫХОД ДС"
- board text added: "Земля"
- board text added: "Питание"
- board text added: "Сигнал"
