File: navigator.kicad_sch (KiCad schematic)
At the start: 29 parts, among them J101 SWD, J102 3V3, J103 5V, J104 GND, J105 INPUT, J106 5V, J107 GND, U101 STM32G030F6Px, U102 5501

Commit message: wip
Parts:
- removed D101: BZX84Cxx, Package_TO_SOT_SMD:SOT-23, symbol Diode:BZX84Cxx
- removed D102: LED_Small, LED_SMD:LED_1206_3216Metric, symbol Device:LED_Small
- removed U101: STM32G030F6Px, Package_SO:TSSOP-20_4.4x6.5mm_P0.65mm, symbol MCU_ST_STM32G0:STM32G030F6Px
- added D101: LED_Small, LED_SMD:LED_1206_3216Metric, symbol Device:LED_Small
- added D104: D_Schottky_Small, Diode_SMD:D_SOD-323, symbol Device:D_Schottky_Small
- added J108: INPUT, Connector_PinHeader_2.54mm:PinHeader_1x01_P2.54mm_Vertical, symbol Connector_Generic:Conn_01x01
- added JP102: Pu/Pd, Jumper:SolderJumper-3_P1.3mm_Open_RoundedPad1.0x1.5mm, symbol Jumper:SolderJumper_3_Open
- added JP103: debug, Jumper:SolderJumper-2_P1.3mm_Open_Pad1.0x1.5mm, symbol Jumper:SolderJumper_2_Open
- added Q101: 2N7002H, Package_TO_SOT_SMD:SOT-23, symbol Transistor_FET:2N7002H
- added R109, R110: 10K, Resistor_SMD:R_0805_2012Metric, symbol Device:R_Small
- added U103: STM32G030J6Mx, Package_SO:SOIC-8_3.9x4.9mm_P1.27mm, symbol MCU_ST_STM32G0:STM32G030J6Mx
- R104: value 1K -> 10K
- R105: value 1K -> 100
Connections:
- net USART1_TX is gone; now on net USART2_TX: R101.1
- net 3V3: now also JP103.2 (B), Q101.1 (G), R110.2, U103.2 (VDD); no longer R103.1
- net 5V: now also R109.2
- net GND: now also R104.1, D101.1 (K), U103.3 (VSS)
- net INPUT: now also R105.1, U103.6 (PA12/PA10); no longer R104.2
- net SWDCLK: now also U103.8 (PA14/PA15/PB5/PB6)
- net SWDIO: now also U103.7 (PA13)
- net USART1_RX: now also U103.1 (PC14/PB7/PB8/PB9)
- net USART2_TX: now also U103.4 (NRST/PA0/PA1/PA2)
- net at R103.2: now also D101.2 (A)
- net at R105.2: now also Q101.2 (S), R110.1
- new net: J108.1 (Pin_1), Q101.3 (D), R109.1
- new net: JP103.1 (A), R103.1, U103.5 (PB0/PB1/PA8/PA11/PA9)
- new net: JP102.1 (A), R104.2
- new net: D104.1 (K), J105.1 (Pin_1), JP102.2 (C)
- new net: JP102.3 (B), R106.1
Other:
- moved on the sheet: C101, J105, R103, R106

Commit message: Production ready
Parts:
- removed D104: D_Schottky_Small, Diode_SMD:D_SOD-323, symbol Device:D_Schottky_Small
- removed J108: INPUT, Connector_PinHeader_2.54mm:PinHeader_1x01_P2.54mm_Vertical, symbol Connector_Generic:Conn_01x01
- removed JP102: Pu/Pd, Jumper:SolderJumper-3_P1.3mm_Open_RoundedPad1.0x1.5mm, symbol Jumper:SolderJumper_3_Open
- removed Q101: 2N7002H, Package_TO_SOT_SMD:SOT-23, symbol Transistor_FET:2N7002H
- removed R110: 10K, Resistor_SMD:R_0805_2012Metric, symbol Device:R_Small
- removed U102: 5501, Package_TO_SOT_SMD:TO-252-3_TabPin2, symbol ncp5500:5501
- added C106: 1uF, Capacitor_SMD:C_0805_2012Metric, symbol Device:C_Small
- added C107, C108: 10uF, Capacitor_SMD:C_0805_2012Metric, symbol Device:C_Small
- added C109: 0.01uF, Capacitor_SMD:C_0603_1608Metric, symbol Device:C_Small
- added D102: SS14FL, Diode_SMD:D_SMF, symbol Device:D_Schottky_Small
- added D104: BZT52C16S, Diode_SMD:D_SOD-323, symbol Device:D_Zener_Small
- added L101: 22uH, inductor:FNR5040S220MT, symbol Device:L_Small
- added LOGO101: ~, logo:logo_15x9, symbol logo:logo
- added Q101: IRLML9303TRPBF, Package_TO_SOT_SMD:SOT-23, symbol Transistor_FET:AO3401A
- added R111: 500, Resistor_SMD:R_0805_2012Metric, symbol Device:R_Small
- added R112: 10K, Resistor_SMD:R_0805_2012Metric, symbol Device:R_Small
- added R113: 200, Resistor_SMD:R_0805_2012Metric, symbol Device:R_Small
- added U101: LTV-817S, Package_DIP:SMDIP-4_W9.53mm, symbol Isolator:LTV-817S
- added U102: LMR16006Y, Package_TO_SOT_SMD:SOT-23-6, symbol Regulator_Switching:LMR16006YQ
- C104: LCSC (none) -> C440198
- C105: value 4.7uF -> 0.1uF; LCSC (none) -> C14663
- J103: value 5V -> Vinn
- J106: value 5V -> SensorV
- R104: value 10K -> 100K; footprint Resistor_SMD:R_0805_2012Metric -> Resistor_SMD:R_0603_1608Metric; LCSC (none) -> C163504
- R105: value 100 -> 28K; footprint Resistor_SMD:R_0805_2012Metric -> Resistor_SMD:R_0603_1608Metric; LCSC (none) -> C728593
- R106: value 10K -> 8K45; footprint Resistor_SMD:R_0805_2012Metric -> Resistor_SMD:R_0603_1608Metric; LCSC (none) -> C98220
- R109: footprint Resistor_SMD:R_0805_2012Metric -> Resistor_SMD:R_0603_1608Metric
Connections:
- net 3V3: now also R105.1, C106.1, C107.1, C108.1, L101.2; no longer C105.1
- net GND: now also R106.2, R109.2, C106.2, C107.2, C108.2, C109.2, D102.2 (A), U101.3, U102.2 (GND); no longer C105.2, R104.1
- net at R105.2: now also R106.1, U102.3 (FB)
- net at R109.1: now also C109.1, D104.2 (A), Q101.1 (G)
- net at JP103.1 (A), R103.1: now also U103.6 (PA12/PA10); no longer U103.5 (PB0/PB1/PA8/PA11/PA9)
- net at R104.2: now also U102.4 (~{SHDN})
- net at J105.1 (Pin_1): now also R112.2, U101.2
- removed net 5V: C104.1, J103.1 (Pin_1), J106.1 (Pin_1), R106.2, R109.2
- removed net INPUT: R105.1, U103.6 (PA12/PA10)
- new net: C105.1, U102.1 (CB)
- new net: C105.2, D102.1 (K), L101.1, U102.6 (SW)
- new net: J103.1 (Pin_1), Q101.3 (D)
- new net: R113.2, U101.4
- new net: R111.2, R112.1, U101.1
- new net SIGNAL: R113.1, U103.5 (PB0/PB1/PA8/PA11/PA9)
- new net Vin: C104.1, D104.1 (K), J106.1 (Pin_1), Q101.2 (S), R104.1, R111.1, U102.5 (VIN)
Other:
- note added: "Input"
- moved on the sheet: D101, J103, J104, J105, J106, J107, JP103, R103
